File: mcp7940n_adapter.kicad_pcb (KiCad board)
At the start: 2 copper layers, 24.1 x 23.5 mm, 7 parts, among them J1 Conn_01x03, J2 Conn_01x02, U1 MCP7940N-xSN, Y1 7pF CL

Commit message: Add attribution and date
Other:
- board text added: "WM v0.0.0 04/07/20"
Changed lines of the file:
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@@
   (general
     (thickness 1.6)
-    (drawings 9)
+    (drawings 10)
     (tracks 41)
     (zones 0)
@@
     (solder_mask_min_width 0.25)
     (aux_axis_origin 0 0)
-    (visible_elements FFFFFF7F)
+    (visible_elements 7FFFFFFF)
     (pcbplotparams
       (layerselection 0x010fc_ffffffff)
@@
     )
   )
+  (gr_text "WM v0.0.0\n04/07/20" (at 144.272 102.616) (layer B.SilkS)
+    (effects (font (size 1.5 1.5) (thickness 0.3)) (justify mirror))
+  )
   (gr_text SCL (at 137.16 86.868 270) (layer F.SilkS)
